File: babble.sch (KiCad schematic (older format))
At the start: 18 parts, among them SW1 power, U1 PIC10F322-IP

Commit message: Projet complété.
Parts:
- removed C2: 10µF, symbol Device:CP
- removed C6: 1n8, symbol Device:C
- removed D2: 1N34, symbol pspice:DIODE
- removed R3, R?: 470, symbol Device:R
- removed R4: 100K, symbol Device:R
- added C2: 1µF, symbol Device:C
Connections:
- net +3volt: now also C2.1
- net GND: now also C2.2
- net PGDAT: now also AE1.1 (A)
- net ~RST: now also C3.2, R2.2
Other:
- moved on the sheet: AE1, BT1, C1, C3, C4, C5, D1, LS1, R1, R2, SW1, U1
